Commit message: first_init

File: simulation_env/autorally_description/urdf/autoRallyPlatform.urdf copy.xacro (robot description, xacro)
@@ -225,6 +225,5 @@
         <origin xyz="0 0 0"/>
         <geometry>
-          <!-- <mesh filename="${wheel_model}" /> -->
-          <cylinder length="0.1" radius="0.09"/>
+          <mesh filename="${wheel_model}" />
         </geometry>
       </collision>
@@ -232,6 +231,5 @@
         <origin xyz="0 0 0"/>
         <geometry>
-          <!-- <mesh filename="${wheel_model}" /> -->
-          <cylinder length="0.1" radius="0.09"/>
+          <mesh filename="${wheel_model}" />
         </geometry>
       </collision>
@@ -336,6 +334,5 @@
               rpy="0 0 0"/>
       <geometry>
-        <!-- <mesh filename="package://autorally_description/urdf/cad/Vehicle_Texture.dae" scale="1 1 1" /> -->
-        <box size="0.01 0.01 0.01"/>
+        <mesh filename="package://autorally_description/urdf/cad/Vehicle_Texture.dae" scale="1 1 1" />
       </geometry>
     </collision>
