Commit message: Camera Projection has bug about near object

File: simulation_env/autorally_description/urdf/autoRallyPlatform.urdf.xacro (robot description, xacro)
@@ -485,4 +485,14 @@
     </inertial>
   </link>
+<joint name="camera_optical_joint" type="fixed">
+    <!-- these values have to be these values otherwise the gazebo camera
+        image won't be aligned properly with the frame it is supposedly
+        originating from -->
+    <origin xyz="0 0 0" rpy="${-pi/2} 0 ${-pi/2}"/>
+    <parent link="camera_link"/>
+    <child link="left_camera_optical_frame"/>
+  </joint>
+  <link name="left_camera_optical_frame">
+  </link>
   <!-- camera -->
   <gazebo reference="camera_link">
@@ -528,5 +538,5 @@
         <robotNamespace>$(arg prefix)</robotNamespace>
         <alwaysOn>true</alwaysOn>
-        <updateRate>60.0</updateRate>
+        <updateRate>30.0</updateRate>
         <cameraName>camera</cameraName>
         <imageTopicName>image_raw</imageTopicName>
